File: main_board/mini_ble.kicad_pcb (KiCad board)
At the start: 4 copper layers, 74.8 x 31.2 mm, 127 parts, among them J1 FIX_M1.4, J2 FIX_M1.4, J4 FIX_M1.4, J7 FIX_M1.4, Q1 SI1013X, Q2 DMN1019USN, Q3 SI1013X, Q4 DMN1019USN, Q5 DMN1019USN, Q6 SI1013X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

Commit message: updated
Connections:
- net /Main MCU & OLED/~RST renamed /Main MCU & OLED/~{RST}
Other:
- net class Default removed
